Commit message: Update (Unsaved).xacro
Updated

File: URDF/(Unsaved)_description/urdf/(Unsaved).xacro (robot description, xacro)
@@ -6,5 +6,5 @@
 <link name="base_link">
   <inertial>
-    <origin xyz="6.436791772353176e-13 8.688569771855988e-06 0.01850253689622171" rpy="0 0 0"/>
+    <origin xyz="6.436791772353176e-13 8.68856977186487e-06 0.08813353689622172" rpy="0 0 0"/>
     <mass value="4.063687233537527"/>
     <inertia ixx="0.025602" iyy="0.025607" izz="0.049318" ixy="0.0" iyz="-0.0" ixz="0.0"/>
@@ -26,10 +26,10 @@
 <link name="Coxa_6">
   <inertial>
-    <origin xyz="-0.020352080722285476 -0.011750115472622377 0.013999999896139464" rpy="0 0 0"/>
+    <origin xyz="-0.020352080722285504 -0.011750115472622377 -0.05563100010386053" rpy="0 0 0"/>
     <mass value="0.09724812532903056"/>
     <inertia ixx="2.5e-05" iyy="3e-05" izz="3.2e-05" ixy="-4e-06" iyz="0.0" ixz="0.0"/>
   </inertial>
   <visual>
-    <origin xyz="0.137878 0.079604 -0.0045" rpy="0 0 0"/>
+    <origin xyz="0.137878 0.079604 -0.143762" rpy="0 0 0"/>
     <geometry>
       <mesh filename="package://(Unsaved)_description/meshes/Coxa_6.stl" scale="0.001 0.001 0.001"/>
@@ -38,5 +38,5 @@
   </visual>
   <collision>
-    <origin xyz="0.137878 0.079604 -0.0045" rpy="0 0 0"/>
+    <origin xyz="0.137878 0.079604 -0.143762" rpy="0 0 0"/>
     <geometry>
       <mesh filename="package://(Unsaved)_description/meshes/Coxa_6.stl" scale="0.001 0.001 0.001"/>
@@ -46,10 +46,10 @@
 <link name="Coxa_1">
   <inertial>
-    <origin xyz="-5.562159473667652e-08 -0.023500327284672773 0.013999999896139467" rpy="0 0 0"/>
+    <origin xyz="-5.562159473445608e-08 -0.023500327284672773 -0.05563100010386053" rpy="0 0 0"/>
     <mass value="0.09724812532903056"/>
     <inertia ixx="3.2e-05" iyy="2.2e-05" izz="3.2e-05" ixy="0.0" iyz="0.0" ixz="-0.0"/>
   </inertial>
   <visual>
-    <origin xyz="-0.0 0.159208 -0.0045" rpy="0 0 0"/>
+    <origin xyz="-0.0 0.159208 -0.143762" rpy="0 0 0"/>
     <geometry>
       <mesh filename="package://(Unsaved)_description/meshes/Coxa_1.stl" scale="0.001 0.001 0.001"/>
@@ -58,5 +58,5 @@
   </visual>
   <collision>
-    <origin xyz="-0.0 0.159208 -0.0045" rpy="0 0 0"/>
+    <origin xyz="-0.0 0.159208 -0.143762" rpy="0 0 0"/>
     <geometry>
       <mesh filename="package://(Unsaved)_description/meshes/Coxa_1.stl" scale="0.001 0.001 0.001"/>
@@ -66,10 +66,10 @@
 <link name="Coxa_2">
   <inertial>
-    <origin xyz="0.0203520251006907 -0.011750211812050437 0.013999999896139464" rpy="0 0 0"/>
+    <origin xyz="0.02350045593286834 -2.1922543673447148e-07 -0.05563100010386053" rpy="0 0 0"/>
     <mass value="0.09724812532903056"/>
-    <inertia ixx="2.5e-05" iyy="3e-05" izz="3.2e-05" ixy="4e-06" iyz="0.0" ixz="-0.0"/>
-  </inertial>
-  <visual>
-    <origin xyz="-0.137878 0.079604 -0.0045" rpy="0 0 0"/>
+    <inertia ixx="2.2e-05" iyy="3.2e-05" izz="3.2e-05" ixy="-0.0" iyz="-0.0" ixz="-0.0"/>
+  </inertial>
+  <visual>
+    <origin xyz="-0.137878 0.079604 -0.143762" rpy="0 0 0"/>
     <geometry>
       <mesh filename="package://(Unsaved)_description/meshes/Coxa_2.stl" scale="0.001 0.001 0.001"/>
@@ -78,5 +78,5 @@
   </visual>
   <collision>
-    <origin xyz="-0.137878 0.079604 -0.0045" rpy="0 0 0"/>
+    <origin xyz="-0.137878 0.079604 -0.143762" rpy="0 0 0"/>
     <geometry>
       <mesh filename="package://(Unsaved)_description/meshes/Coxa_2.stl" scale="0.001 0.001 0.001"/>
@@ -86,10 +86,10 @@
 <link name="Coxa_3">
   <inertial>
-    <origin xyz="0.02035208072228556 0.011750115472622377 0.013999999896139464" rpy="0 0 0"/>
+    <origin xyz="0.02035208072228556 0.011750115472622377 -0.05563100010386053" rpy="0 0 0"/>
     <mass value="0.09724812532903056"/>
     <inertia ixx="2.5e-05" iyy="3e-05" izz="3.2e-05" ixy="-4e-06" iyz="-0.0" ixz="-0.0"/>
   </inertial>
   <visual>
-    <origin xyz="-0.137878 -0.079604 -0.0045" rpy="0 0 0"/>
+    <origin xyz="-0.137878 -0.079604 -0.143762" rpy="0 0 0"/>
     <geometry>
       <mesh filename="package://(Unsaved)_description/meshes/Coxa_3.stl" scale="0.001 0.001 0.001"/>
@@ -98,5 +98,5 @@
   </visual>
   <collision>
-    <origin xyz="-0.137878 -0.079604 -0.0045" rpy="0 0 0"/>
+    <origin xyz="-0.137878 -0.079604 -0.143762" rpy="0 0 0"/>
     <geometry>
       <mesh filename="package://(Unsaved)_description/meshes/Coxa_3.stl" scale="0.001 0.001 0.001"/>
@@ -106,10 +106,10 @@
 <link name="Coxa_4">
   <inertial>
-    <origin xyz="5.562159476619979e-08 0.023500327284672745 0.013999999896139467" rpy="0 0 0"/>
+    <origin xyz="5.562159475807144e-08 0.02350032728467269 -0.05563100010386053" rpy="0 0 0"/>
     <mass value="0.09724812532903056"/>
     <inertia ixx="3.2e-05" iyy="2.2e-05" izz="3.2e-05" ixy="0.0" iyz="-0.0" ixz="0.0"/>
   </inertial>
   <visual>
-    <origin xyz="-0.0 -0.159208 -0.0045" rpy="0 0 0"/>
+    <origin xyz="-0.0 -0.159208 -0.143762" rpy="0 0 0"/>
     <geometry>
       <mesh filename="package://(Unsaved)_description/meshes/Coxa_4.stl" scale="0.001 0.001 0.001"/>
@@ -118,5 +118,5 @@
   </visual>
   <collision>
-    <origin xyz="-0.0 -0.159208 -0.0045" rpy="0 0 0"/>
+    <origin xyz="-0.0 -0.159208 -0.143762" rpy="0 0 0"/>
     <geometry>
       <mesh filename="package://(Unsaved)_description/meshes/Coxa_4.stl" scale="0.001 0.001 0.001"/>
@@ -126,10 +126,10 @@
 <link name="Coxa_5">
   <inertial>
-    <origin xyz="-0.0203520251006907 0.011750211812050507 0.013999999896139464" rpy="0 0 0"/>
+    <origin xyz="-0.02350045593286834 2.1922543678998263e-07 -0.05563100010386053" rpy="0 0 0"/>
     <mass value="0.09724812532903056"/>
-    <inertia ixx="2.5e-05" iyy="3e-05" izz="3.2e-05" ixy="4e-06" iyz="-0.0" ixz="0.0"/>
-  </inertial>
-  <visual>
-    <origin xyz="0.137878 -0.079604 -0.0045" rpy="0 0 0"/>
+    <inertia ixx="2.2e-05" iyy="3.2e-05" izz="3.2e-05" ixy="-0.0" iyz="0.0" ixz="0.0"/>
+  </inertial>
+  <visual>
+    <origin xyz="0.137878 -0.079604 -0.143762" rpy="0 0 0"/>
     <geometry>
       <mesh filename="package://(Unsaved)_description/meshes/Coxa_5.stl" scale="0.001 0.001 0.001"/>
@@ -138,5 +138,5 @@
   </visual>
   <collision>
-    <origin xyz="0.137878 -0.079604 -0.0045" rpy="0 0 0"/>
+    <origin xyz="0.137878 -0.079604 -0.143762" rpy="0 0 0"/>
     <geometry>
       <mesh filename="package://(Unsaved)_description/meshes/Coxa_5.stl" scale="0.001 0.001 0.001"/>
@@ -146,10 +146,10 @@
 <link name="Femur_2">
   <inertial>
-    <origin xyz="0.031755805786388674 -0.21617124089933584 -0.0011332936485353023" rpy="0 0 0"/>
+    <origin xyz="0.15714461044686726 -0.18487816360384196 -0.0707642936485353" rpy="0 0 0"/>
     <mass value="0.18493846398077138"/>
-    <inertia ixx="3.3e-05" iyy="4.4e-05" izz="6e-05" ixy="1e-05" iyz="-3e-06" ixz="5e-06"/>
-  </inertial>
-  <visual>
-    <origin xyz="-0.159851 -0.105547 -0.0185" rpy="0 0 0"/>
+    <inertia ixx="2.8e-05" iyy="5e-05" izz="6e-05" ixy="0.0" iyz="-0.0" ixz="6e-06"/>
+  </inertial>
+  <visual>
+    <origin xyz="-0.042774 -0.105274 -0.157762" rpy="0 0 0"/>
     <geometry>
       <mesh filename="package://(Unsaved)_description/meshes/Femur_2.stl" scale="0.001 0.001 0.001"/>
@@ -158,5 +158,5 @@
   </visual>
   <collision>
-    <origin xyz="-0.159851 -0.105547 -0.0185" rpy="0 0 0"/>
+    <origin xyz="-0.042774 -0.105274 -0.157762" rpy="0 0 0"/>
     <geometry>
       <mesh filename="package://(Unsaved)_description/meshes/Femur_2.stl" scale="0.001 0.001 0.001"/>
@@ -166,10 +166,10 @@
 <link name="Femur_3">
   <inertial>
-    <origin xyz="0.38891880578638915 0.009962240899335978 -0.0011332936485353093" rpy="0 0 0"/>
+    <origin xyz="0.38891880578638915 0.009962240899335978 -0.07076429364853531" rpy="0 0 0"/>
     <mass value="0.18493846398077138"/>
     <inertia ixx="3.3e-05" iyy="4.4e-05" izz="6e-05" ixy="-1e-05" iyz="3e-06" ixz="5e-06"/>
   </inertial>
   <visual>
-    <origin xyz="0.197312 -0.100662 -0.0185" rpy="0 0 0"/>
+    <origin xyz="0.197312 -0.100662 -0.157762" rpy="0 0 0"/>
     <geometry>
       <mesh filename="package://(Unsaved)_description/meshes/Femur_3.stl" scale="0.001 0.001 0.001"/>
@@ -178,5 +178,5 @@
   </visual>
   <collision>
-    <origin xyz="0.197312 -0.100662 -0.0185" rpy="0 0 0"/>
+    <origin xyz="0.197312 -0.100662 -0.157762" rpy="0 0 0"/>
     <geometry>
       <mesh filename="package://(Unsaved)_description/meshes/Femur_3.stl" scale="0.001 0.001 0.001"/>
@@ -186,10 +186,10 @@
 <link name="Femur_4">
   <inertial>
-    <origin xyz="0.014500000000000065 0.45745648179867177 -0.0011332936485352989" rpy="0 0 0"/>
+    <origin xyz="0.01450000000000005 0.45745648179867177 -0.0707642936485353" rpy="0 0 0"/>
     <mass value="0.18493846398077138"/>
     <inertia ixx="5e-05" iyy="2.8e-05" izz="6e-05" ixy="-0.0" iyz="6e-06" ixz="0.0"/>
   </inertial>
   <visual>
-    <origin xyz="0.0145 0.236208 -0.0185" rpy="0 0 0"/>
+    <origin xyz="0.0145 0.236208 -0.157762" rpy="0 0 0"/>
     <geometry>
       <mesh filename="package://(Unsaved)_description/meshes/Femur_4.stl" scale="0.001 0.001 0.001"/>
@@ -198,5 +198,5 @@
   </visual>
   <collision>
-    <origin xyz="0.0145 0.236208 -0.0185" rpy="0 0 0"/>
+    <origin xyz="0.0145 0.236208 -0.157762" rpy="0 0 0"/>
     <geometry>
       <mesh filename="package://(Unsaved)_description/meshes/Femur_4.stl" scale="0.001 0.001 0.001"/>
@@ -206,10 +206,10 @@
 <link name="Femur_5">
   <inertial>
-    <origin xyz="-0.40341880578638867 0.03507724089933596 -0.0011332936485353023" rpy="0 0 0"/>
+    <origin xyz="-0.3453526104468674 -0.184878836396158 -0.0707642936485353" rpy="0 0 0"/>
     <mass value="0.18493846398077138"/>
-    <inertia ixx="3.3e-05" iyy="4.4e-05" izz="6e-05" ixy="1e-05" iyz="3e-06" ixz="-5e-06"/>
-  </inertial>
-  <visual>
-    <origin xyz="-0.211812 -0.075547 -0.0185" rpy="0 0 0"/>
+    <inertia ixx="2.8e-05" iyy="5e-05" izz="6e-05" ixy="0.0" iyz="0.0" ixz="-6e-06"/>
+  </inertial>
+  <visual>
+    <origin xyz="-0.145434 -0.264483 -0.157762" rpy="0 0 0"/>
     <geometry>
       <mesh filename="package://(Unsaved)_description/meshes/Femur_5.stl" scale="0.001 0.001 0.001"/>
@@ -218,5 +218,5 @@
   </visual>
   <collision>
-    <origin xyz="-0.211812 -0.075547 -0.0185" rpy="0 0 0"/>
+    <origin xyz="-0.145434 -0.264483 -0.157762" rpy="0 0 0"/>
     <geometry>
       <mesh filename="package://(Unsaved)_description/meshes/Femur_5.stl" scale="0.001 0.001 0.001"/>
@@ -226,10 +226,10 @@
 <link name="Femur_6">
   <inertial>
-    <origin xyz="-0.03175580578638865 -0.2161712408993359 -0.0011332936485353023" rpy="0 0 0"/>
+    <origin xyz="-0.03175580578638865 -0.2161712408993359 -0.0707642936485353" rpy="0 0 0"/>
     <mass value="0.18493846398077138"/>
     <inertia ixx="3.3e-05" iyy="4.4e-05" izz="6e-05" ixy="-1e-05" iyz="-3e-06" ixz="-5e-06"/>
   </inertial>
   <visual>
-    <origin xyz="0.159851 -0.105547 -0.0185" rpy="0 0 0"/>
+    <origin xyz="0.159851 -0.105547 -0.157762" rpy="0 0 0"/>
     <geometry>
       <mesh filename="package://(Unsaved)_description/meshes/Femur_6.stl" scale="0.001 0.001 0.001"/>
@@ -238,5 +238,5 @@
   </visual>
   <collision>
-    <origin xyz="0.159851 -0.105547 -0.0185" rpy="0 0 0"/>
+    <origin xyz="0.159851 -0.105547 -0.157762" rpy="0 0 0"/>
     <geometry>
       <mesh filename="package://(Unsaved)_description/meshes/Femur_6.stl" scale="0.001 0.001 0.001"/>
@@ -246,10 +246,10 @@
 <link name="Femur_1">
   <inertial>
-    <origin xyz="0.014499999999999978 -0.04504048179867179 -0.0011332936485352989" rpy="0 0 0"/>
+    <origin xyz="0.014499999999999985 -0.04504048179867179 -0.0707642936485353" rpy="0 0 0"/>
     <mass value="0.18493846398077138"/>
     <inertia ixx="5e-05" iyy="2.8e-05" izz="6e-05" ixy="-0.0" iyz="-6e-06" ixz="-0.0"/>
   </inertial>
   <visual>
-    <origin xyz="0.0145 0.176208 -0.0185" rpy="0 0 0"/>
+    <origin xyz="0.0145 0.176208 -0.157762" rpy="0 0 0"/>
     <geometry>
       <mesh filename="package://(Unsaved)_description/meshes/Femur_1.stl" scale="0.001 0.001 0.001"/>
@@ -258,5 +258,5 @@
   </visual>
   <collision>
-    <origin xyz="0.0145 0.176208 -0.0185" rpy="0 0 0"/>
+    <origin xyz="0.0145 0.176208 -0.157762" rpy="0 0 0"/>
     <geometry>
       <mesh filename="package://(Unsaved)_description/meshes/Femur_1.stl" scale="0.001 0.001 0.001"/>
@@ -266,10 +266,10 @@
 <link name="Tibia_3">
   <inertial>
-    <origin xyz="0.509230767163375 0.03563522060723821 -0.016307916271994807" rpy="0 0 0"/>
+    <origin xyz="0.509230767163375 0.03563522060723821 -0.08593891627199479" rpy="0 0 0"/>
     <mass value="0.25344458673845177"/>
     <inertia ixx="0.000236" iyy="0.000295" izz="0.000178" ixy="-5.2e-05" iyz="7e-05" ixz="0.000122"/>
   </inertial>
   <visual>
-    <origin xyz="0.269376 -0.102845 -0.005074" rpy="0 0 0"/>
+    <origin xyz="0.269376 -0.102845 -0.144336" rpy="0 0 0"/>
     <geometry>
       <mesh filename="package://(Unsaved)_description/meshes/Tibia_3.stl" scale="0.001 0.001 0.001"/>
@@ -278,5 +278,5 @@
   </visual>
   <collision>
-    <origin xyz="0.269376 -0.102845 -0.005074" rpy="0 0 0"/>
+    <origin xyz="0.269376 -0.102845 -0.144336" rpy="0 0 0"/>
     <geometry>
       <mesh filename="package://(Unsaved)_description/meshes/Tibia_3.stl" scale="0.001 0.001 0.001"/>
@@ -286,10 +286,10 @@
 <link name="Tibia_4">
   <inertial>
-    <origin xyz="0.01499999461414578 0.5966684318859028 -0.0163079162719948" rpy="0 0 0"/>
+    <origin xyz="0.01499999461414578 0.5966684318859028 -0.08593891627199479" rpy="0 0 0"/>
     <mass value="0.25344458673845177"/>
     <inertia ixx="0.000325" iyy="0.000206" izz="0.000178" ixy="0.0" iyz="0.00014" ixz="0.0"/>
   </inertial>
   <visual>
-    <origin xyz="0.015 0.319708 -0.005074" rpy="0 0 0"/>
+    <origin xyz="0.015 0.319708 -0.144336" rpy="0 0 0"/>
     <geometry>
       <mesh filename="package://(Unsaved)_description/meshes/Tibia_4.stl" scale="0.001 0.001 0.001"/>
@@ -298,5 +298,5 @@
   </visual>
   <collision>
-    <origin xyz="0.015 0.319708 -0.005074" rpy="0 0 0"/>
+    <origin xyz="0.015 0.319708 -0.144336" rpy="0 0 0"/>
     <geometry>
       <mesh filename="package://(Unsaved)_description/meshes/Tibia_4.stl" scale="0.001 0.001 0.001"/>
@@ -306,10 +306,10 @@
 <link name="Tibia_5">
   <inertial>
-    <origin xyz="-0.5242307725492287 0.061616211278664804 -0.016307916271994797" rpy="0 0 0"/>
+    <origin xyz="-0.4415645605340984 -0.22837884178201232 -0.08593891627199479" rpy="0 0 0"/>
     <mass value="0.25344458673845177"/>
-    <inertia ixx="0.000236" iyy="0.000295" izz="0.000178" ixy="5.2e-05" iyz="7e-05" ixz="-0.000122"/>
-  </inertial>
-  <visual>
-    <origin xyz="-0.284376 -0.076864 -0.005074" rpy="0 0 0"/>
+    <inertia ixx="0.000206" iyy="0.000325" izz="0.000178" ixy="-0.0" iyz="0.0" ixz="-0.00014"/>
+  </inertial>
+  <visual>
+    <origin xyz="-0.185934 -0.307983 -0.144336" rpy="0 0 0"/>
     <geometry>
       <mesh filename="package://(Unsaved)_description/meshes/Tibia_5.stl" scale="0.001 0.001 0.001"/>
@@ -318,5 +318,5 @@
   </visual>
   <collision>
-    <origin xyz="-0.284376 -0.076864 -0.005074" rpy="0 0 0"/>
+    <origin xyz="-0.185934 -0.307983 -0.144336" rpy="0 0 0"/>
     <geometry>
       <mesh filename="package://(Unsaved)_description/meshes/Tibia_5.stl" scale="0.001 0.001 0.001"/>
@@ -326,10 +326,10 @@
 <link name="Tibia_6">
   <inertial>
-    <origin xyz="-0.09172276716337444 -0.3113252206072381 -0.0163079162719948" rpy="0 0 0"/>
+    <origin xyz="-0.09172276716337444 -0.3113252206072381 -0.08593891627199479" rpy="0 0 0"/>
     <mass value="0.25344458673845177"/>
     <inertia ixx="0.000236" iyy="0.000295" izz="0.000178" ixy="-5.2e-05" iyz="-7e-05" ixz="-0.000122"/>
   </inertial>
   <visual>
-    <origin xyz="0.148132 -0.172845 -0.005074" rpy="0 0 0"/>
+    <origin xyz="0.148132 -0.172845 -0.144336" rpy="0 0 0"/>
     <geometry>
       <mesh filename="package://(Unsaved)_description/meshes/Tibia_6.stl" scale="0.001 0.001 0.001"/>
@@ -338,5 +338,5 @@
   </visual>
   <collision>
-    <origin xyz="0.148132 -0.172845 -0.005074" rpy="0 0 0"/>
+    <origin xyz="0.148132 -0.172845 -0.144336" rpy="0 0 0"/>
     <geometry>
       <mesh filename="package://(Unsaved)_description/meshes/Tibia_6.stl" scale="0.001 0.001 0.001"/>
@@ -346,10 +346,10 @@
 <link name="Tibia_1">
   <inertial>
-    <origin xyz="0.01500000538585427 -0.09725243188590285 -0.0163079162719948" rpy="0 0 0"/>
+    <origin xyz="0.015000005385854264 -0.09725243188590285 -0.08593891627199479" rpy="0 0 0"/>
     <mass value="0.25344458673845177"/>
     <inertia ixx="0.000325" iyy="0.000206" izz="0.000178" ixy="0.0" iyz="-0.00014" ixz="-0.0"/>
   </inertial>
   <visual>
-    <origin xyz="0.015 0.179708 -0.005074" rpy="0 0 0"/>
+    <origin xyz="0.015 0.179708 -0.144336" rpy="0 0 0"/>
     <geometry>
       <mesh filename="package://(Unsaved)_description/meshes/Tibia_1.stl" scale="0.001 0.001 0.001"/>
@@ -358,5 +358,5 @@
   </visual>
   <collision>
-    <origin xyz="0.015 0.179708 -0.005074" rpy="0 0 0"/>
+    <origin xyz="0.015 0.179708 -0.144336" rpy="0 0 0"/>
     <geometry>
       <mesh filename="package://(Unsaved)_description/meshes/Tibia_1.stl" scale="0.001 0.001 0.001"/>
@@ -366,10 +366,10 @@
 <link name="Tibia_2">
   <inertial>
-    <origin xyz="0.0767227725492286 -0.28534421127866466 -0.016307916271994797" rpy="0 0 0"/>
+    <origin xyz="0.25235656053409833 -0.2283781582179876 -0.08593891627199479" rpy="0 0 0"/>
     <mass value="0.25344458673845177"/>
-    <inertia ixx="0.000236" iyy="0.000295" izz="0.000178" ixy="5.2e-05" iyz="-7e-05" ixz="0.000122"/>
-  </inertial>
-  <visual>
-    <origin xyz="-0.163132 -0.146864 -0.005074" rpy="0 0 0"/>
+    <inertia ixx="0.000206" iyy="0.000325" izz="0.000178" ixy="-0.0" iyz="-0.0" ixz="0.00014"/>
+  </inertial>
+  <visual>
+    <origin xyz="-0.003274 -0.148774 -0.144336" rpy="0 0 0"/>
     <geometry>
       <mesh filename="package://(Unsaved)_description/meshes/Tibia_2.stl" scale="0.001 0.001 0.001"/>
@@ -378,5 +378,5 @@
   </visual>
   <collision>
-    <origin xyz="-0.163132 -0.146864 -0.005074" rpy="0 0 0"/>
+    <origin xyz="-0.003274 -0.148774 -0.144336" rpy="0 0 0"/>
     <geometry>
       <mesh filename="package://(Unsaved)_description/meshes/Tibia_2.stl" scale="0.001 0.001 0.001"/>
@@ -385,50 +385,50 @@
 </link>
 <joint name="Revolute 1" type="revolute">
-  <origin xyz="-0.137878 -0.079604 0.0045" rpy="0 0 0"/>
+  <origin xyz="-0.137878 -0.079604 0.143762" rpy="0 0 0"/>
   <parent link="base_link"/>
   <child link="Coxa_6"/>
-  <axis xyz="0.0 0.0 1.0"/>
+  <axis xyz="-0.0 -0.0 1.0"/>
   <limit upper="1.570796" lower="-1.570796" effort="100" velocity="100"/>
 </joint>
 <joint name="Revolute 2" type="revolute">
-  <origin xyz="0.0 -0.159208 0.0045" rpy="0 0 0"/>
+  <origin xyz="0.0 -0.159208 0.143762" rpy="0 0 0"/>
   <parent link="base_link"/>
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