Commit message: Made file paths relative in URDF

File: meshcat_sim/hexy_urdf_v2_dae/hexy_urdf_v2.urdf (robot description, URDF)
Before this commit: robot base_link, 19 links, 18 joints
Links:
- link Coxa_1: geometry visual mesh filename=file://hexy_urdf_v2_dae/hexy_urdf_v2_Coxa_1_vis_1.dae
- link Coxa_2: geometry visual mesh filename=file://hexy_urdf_v2_dae/hexy_urdf_v2_Coxa_2_vis_1.dae
- link Coxa_3: geometry visual mesh filename=file://hexy_urdf_v2_dae/hexy_urdf_v2_Coxa_3_vis_1.dae
- link Coxa_4: geometry visual mesh filename=file://hexy_urdf_v2_dae/hexy_urdf_v2_Coxa_4_vis_1.dae
- link Coxa_5: geometry visual mesh filename=file://hexy_urdf_v2_dae/hexy_urdf_v2_Coxa_5_vis_1.dae
- link Coxa_6: geometry visual mesh filename=file://hexy_urdf_v2_dae/hexy_urdf_v2_Coxa_6_vis_1.dae
- link Femur_1: geometry visual mesh filename=file://hexy_urdf_v2_dae/hexy_urdf_v2_Femur_1_vis_1.dae
- link Femur_2: geometry visual mesh filename=file://hexy_urdf_v2_dae/hexy_urdf_v2_Femur_2_vis_1.dae
- link Femur_3: geometry visual mesh filename=file://hexy_urdf_v2_dae/hexy_urdf_v2_Femur_3_vis_1.dae
- link Femur_4: geometry visual mesh filename=file://hexy_urdf_v2_dae/hexy_urdf_v2_Femur_4_vis_1.dae
- link Femur_5: geometry visual mesh filename=file://hexy_urdf_v2_dae/hexy_urdf_v2_Femur_5_vis_1.dae
- link Femur_6: geometry visual mesh filename=file://hexy_urdf_v2_dae/hexy_urdf_v2_Femur_6_vis_1.dae
- link Tibia_1: geometry visual mesh filename=file://hexy_urdf_v2_dae/hexy_urdf_v2_Tibia_1_vis_1.dae
- link Tibia_2: geometry visual mesh filename=file://hexy_urdf_v2_dae/hexy_urdf_v2_Tibia_2_vis_1.dae
- link Tibia_3: geometry visual mesh filename=file://hexy_urdf_v2_dae/hexy_urdf_v2_Tibia_3_vis_1.dae
- link Tibia_4: geometry visual mesh filename=file://hexy_urdf_v2_dae/hexy_urdf_v2_Tibia_4_vis_1.dae
- link Tibia_5: geometry visual mesh filename=file://hexy_urdf_v2_dae/hexy_urdf_v2_Tibia_5_vis_1.dae
- link Tibia_6: geometry visual mesh filename=file://hexy_urdf_v2_dae/hexy_urdf_v2_Tibia_6_vis_1.dae
- link robot_base: geometry visual mesh filename=file://hexy_urdf_v2_dae/hexy_urdf_v2_robot_base_vis_1.dae
