Commit message: Collision handling added

File: meshcat_sim/hexy_urdf_v2_1_1_dae/hexy_urdf_v2_1.urdf (robot description, URDF)
Before this commit: robot base_link, 19 links, 18 joints
Links:
- link Coxa_1: geometry collision mesh filename=file://hexy_urdf_v2_4_dae/hexy_urdf_v2_4_Coxa_1_vis_1.dae; visual mesh filename=file://hexy_urdf_v2_dae/hexy_urdf_v2_Coxa_1_vis_1.dae
- link Coxa_2: geometry collision mesh filename=file://hexy_urdf_v2_4_dae/hexy_urdf_v2_4_Coxa_2_vis_1.dae; visual mesh filename=file://hexy_urdf_v2_dae/hexy_urdf_v2_Coxa_2_vis_1.dae
- link Coxa_3: geometry collision mesh filename=file://hexy_urdf_v2_4_dae/hexy_urdf_v2_4_Coxa_3_vis_1.dae; visual mesh filename=file://hexy_urdf_v2_dae/hexy_urdf_v2_Coxa_3_vis_1.dae
- link Coxa_4: geometry collision mesh filename=file://hexy_urdf_v2_4_dae/hexy_urdf_v2_4_Coxa_4_vis_1.dae; visual mesh filename=file://hexy_urdf_v2_dae/hexy_urdf_v2_Coxa_4_vis_1.dae
- link Coxa_5: geometry collision mesh filename=file://hexy_urdf_v2_4_dae/hexy_urdf_v2_4_Coxa_5_vis_1.dae; visual mesh filename=file://hexy_urdf_v2_dae/hexy_urdf_v2_Coxa_5_vis_1.dae
- link Coxa_6: geometry collision mesh filename=file://hexy_urdf_v2_4_dae/hexy_urdf_v2_4_Coxa_6_vis_1.dae; visual mesh filename=file://hexy_urdf_v2_dae/hexy_urdf_v2_Coxa_6_vis_1.dae
- link Femur_1: geometry collision mesh filename=file://hexy_urdf_v2_4_dae/hexy_urdf_v2_4_Femur_1_vis_1.dae; visual mesh filename=file://hexy_urdf_v2_dae/hexy_urdf_v2_Femur_1_vis_1.dae
- link Femur_2: geometry collision mesh filename=file://hexy_urdf_v2_4_dae/hexy_urdf_v2_4_Femur_2_vis_1.dae; visual mesh filename=file://hexy_urdf_v2_dae/hexy_urdf_v2_Femur_2_vis_1.dae
- link Femur_3: geometry collision mesh filename=file://hexy_urdf_v2_4_dae/hexy_urdf_v2_4_Femur_3_vis_1.dae; visual mesh filename=file://hexy_urdf_v2_dae/hexy_urdf_v2_Femur_3_vis_1.dae
- link Femur_4: geometry collision mesh filename=file://hexy_urdf_v2_4_dae/hexy_urdf_v2_4_Femur_4_vis_1.dae; visual mesh filename=file://hexy_urdf_v2_dae/hexy_urdf_v2_Femur_4_vis_1.dae
- link Femur_5: geometry collision mesh filename=file://hexy_urdf_v2_4_dae/hexy_urdf_v2_4_Femur_5_vis_1.dae; visual mesh filename=file://hexy_urdf_v2_dae/hexy_urdf_v2_Femur_5_vis_1.dae
- link Femur_6: geometry collision mesh filename=file://hexy_urdf_v2_4_dae/hexy_urdf_v2_4_Femur_6_vis_1.dae; visual mesh filename=file://hexy_urdf_v2_dae/hexy_urdf_v2_Femur_6_vis_1.dae
- link Tibia_1: geometry collision mesh filename=file://hexy_urdf_v2_4_dae/hexy_urdf_v2_4_Tibia_1_vis_1.dae; visual mesh filename=file://hexy_urdf_v2_dae/hexy_urdf_v2_Tibia_1_vis_1.dae
- link Tibia_2: geometry collision mesh filename=file://hexy_urdf_v2_4_dae/hexy_urdf_v2_4_Tibia_2_vis_1.dae; visual mesh filename=file://hexy_urdf_v2_dae/hexy_urdf_v2_Tibia_2_vis_1.dae
- link Tibia_3: geometry collision mesh filename=file://hexy_urdf_v2_4_dae/hexy_urdf_v2_4_Tibia_3_vis_1.dae; visual mesh filename=file://hexy_urdf_v2_dae/hexy_urdf_v2_Tibia_3_vis_1.dae
- link Tibia_4: geometry collision mesh filename=file://hexy_urdf_v2_4_dae/hexy_urdf_v2_4_Tibia_4_vis_1.dae; visual mesh filename=file://hexy_urdf_v2_dae/hexy_urdf_v2_Tibia_4_vis_1.dae
- link Tibia_5: geometry collision mesh filename=file://hexy_urdf_v2_4_dae/hexy_urdf_v2_4_Tibia_5_vis_1.dae; visual mesh filename=file://hexy_urdf_v2_dae/hexy_urdf_v2_Tibia_5_vis_1.dae
- link Tibia_6: geometry collision mesh filename=file://hexy_urdf_v2_4_dae/hexy_urdf_v2_4_Tibia_6_vis_1.dae; visual mesh filename=file://hexy_urdf_v2_dae/hexy_urdf_v2_Tibia_6_vis_1.dae
- link robot_base: geometry collision mesh filename=file://hexy_urdf_v2_4_dae/hexy_urdf_v2_4_robot_base_vis_1.d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; visual mesh filename=file://hexy_urdf_v2_dae/hexy_urdf_v2_robot_base_vis_1.dae
Joints:
- joint Revolute_joint: limit lower=-1.0471975511967 upper=1.0471975511967 effort=0.52 velocity=10.786134777326 -> (none); type revolute -> continuous
- joint Revolute_joint_10: limit lower=-1.0471975511967 upper=1.0471975511967 effort=0.52 velocity=10.786134777326 -> (none); type revolute -> continuous
- joint Revolute_joint_11: limit lower=-1.0471975511967 upper=1.0471975511967 effort=0.52 velocity=10.786134777326 -> (none); type revolute -> continuous
- joint Revolute_joint_12: limit lower=-1.0471975511967 upper=1.0471975511967 effort=0.52 velocity=10.786134777326 -> (none); type revolute -> continuous
- joint Revolute_joint_13: limit lower=-1.0471975511967 upper=1.0471975511967 effort=0.52 velocity=10.786134777326 -> (none); type revolute -> continuous
- joint Revolute_joint_14: limit lower=-1.0471975511967 upper=1.0471975511967 effort=0.52 velocity=10.786134777326 -> (none); type revolute -> continuous
- joint Revolute_joint_15: limit lower=-1.0471975511967 upper=1.0471975511967 effort=0.52 velocity=10.786134777326 -> (none); type revolute -> continuous
- joint Revolute_joint_16: limit lower=-1.0471975511967 upper=1.0471975511967 effort=0.52 velocity=10.786134777326 -> (none); type revolute -> continuous
- joint Revolute_joint_17: limit lower=-1.0471975511967 upper=1.0471975511967 effort=0.52 velocity=10.786134777326 -> (none); type revolute -> continuous
- joint Revolute_joint_18: limit lower=-1.0471975511967 upper=1.0471975511967 effort=0.52 velocity=10.786134777326 -> (none); type revolute -> continuous
- joint Revolute_joint_2: limit lower=-1.0471975511967 upper=1.0471975511967 effort=0.52 velocity=10.786134777326 -> (none); type revolute -> continuous
- joint Revolute_joint_3: limit lower=-0.61086523819806 upper=1.4835298641953 effort=0.52 velocity=10.786134777326 -> (none); type revolute -> continuous
- joint Revolute_joint_4: limit lower=-1.0471975511967 upper=1.0471975511967 effort=0.52 velocity=10.786134777326 -> (none); type revolute -> continuous
- joint Revolute_joint_5: limit lower=-1.0471975511967 upper=1.0471975511967 effort=0.52 velocity=10.786134777326 -> (none); type revolute -> continuous
- joint Revolute_joint_6: limit lower=-0.61086523819806 upper=1.4835298641953 effort=0.52 velocity=10.786134777326 -> (none); type revolute -> continuous
- joint Revolute_joint_7: limit lower=-1.0471975511967 upper=1.0471975511967 effort=0.52 velocity=10.786134777326 -> (none); type revolute -> continuous
- joint Revolute_joint_8: limit lower=-1.0471975511967 upper=1.0471975511967 effort=0.52 velocity=10.786134777326 -> (none); type revolute -> continuous
- joint Revolute_joint_9: limit lower=-1.0471975511967 upper=1.0471975511967 effort=0.52 velocity=10.786134777326 -> (none); type revolute -> continuous
