Commit message: URDF Updated (All joints changed from continuous to revolute)

File: meshcat_sim/URDF/URDF4Pin/URDF4Pin.urdf (robot description, URDF)
Before this commit: robot base_link, 25 links, 24 joints
Joints:
- joint Revolute_joint_01: limit (none) -> lower=-1.0471975511967 upper=1.0471975511967 effort=0.52 velocity=10.786134777326; type continuous -> revolute
- joint Revolute_joint_02: limit (none) -> lower=-1.0471975511967 upper=1.0471975511967 effort=0.52 velocity=10.786134777326; type continuous -> revolute
- joint Revolute_joint_03: limit (none) -> lower=-1.0471975511967 upper=1.0471975511967 effort=0.52 velocity=10.786134777326; type continuous -> revolute
- joint Revolute_joint_04: limit (none) -> lower=-1.0471975511967 upper=1.0471975511967 effort=0.52 velocity=10.786134777326; type continuous -> revolute
- joint Revolute_joint_05: limit (none) -> lower=-1.0471975511967 upper=1.0471975511967 effort=0.52 velocity=10.786134777326; type continuous -> revolute
- joint Revolute_joint_06: limit (none) -> lower=-1.0471975511967 upper=1.0471975511967 effort=0.52 velocity=10.786134777326; type continuous -> revolute
- joint Revolute_joint_11: limit (none) -> lower=-1.0471975511967 upper=1.0471975511967 effort=0.52 velocity=10.786134777326; type continuous -> revolute
- joint Revolute_joint_12: limit (none) -> lower=-1.0471975511967 upper=1.0471975511967 effort=0.52 velocity=10.786134777326; type continuous -> revolute
- joint Revolute_joint_13: limit (none) -> lower=-1.0471975511967 upper=1.0471975511967 effort=0.52 velocity=10.786134777326; type continuous -> revolute
- joint Revolute_joint_14: limit (none) -> lower=-1.0471975511967 upper=1.0471975511967 effort=0.52 velocity=10.786134777326; type continuous -> revolute
- joint Revolute_joint_15: limit (none) -> lower=-1.0471975511967 upper=1.0471975511967 effort=0.52 velocity=10.786134777326; type continuous -> revolute
- joint Revolute_joint_16: limit (none) -> lower=-1.0471975511967 upper=1.0471975511967 effort=0.52 velocity=10.786134777326; type continuous -> revolute
- joint Revolute_joint_21: limit (none) -> lower=-1.0471975511967 upper=1.0471975511967 effort=0.52 velocity=10.786134777326; type continuous -> revolute
- joint Revolute_joint_22: limit (none) -> lower=-1.0471975511967 upper=1.0471975511967 effort=0.52 velocity=10.786134777326; type continuous -> revolute
- joint Revolute_joint_23: limit (none) -> lower=-1.0471975511967 upper=1.0471975511967 effort=0.52 velocity=10.786134777326; type continuous -> revolute
- joint Revolute_joint_24: limit (none) -> lower=-1.0471975511967 upper=1.0471975511967 effort=0.52 velocity=10.786134777326; type continuous -> revolute
- joint Revolute_joint_25: limit (none) -> lower=-1.0471975511967 upper=1.0471975511967 effort=0.52 velocity=10.786134777326; type continuous -> revolute
- joint Revolute_joint_26: limit (none) -> lower=-1.0471975511967 upper=1.0471975511967 effort=0.52 velocity=10.786134777326; type continuous -> revolute
- joint Spherical_joint_31: axis 0 0 1 -> (none)

Commit message: 1. Joint names in updated in URDF 2. Foot trajectory logic moved from main to hexapod class

File: meshcat_sim/URDF/URDF4Pin/URDF4Pin.urdf (robot description, URDF)
Before this commit: robot base_link, 25 links, 24 joints
Joints:
- removed joint Spherical_joint_31
- removed joint Spherical_joint_32
- removed joint Spherical_joint_33
- removed joint Spherical_joint_34
- removed joint Spherical_joint_35
- removed joint Spherical_joint_36
- added joint fixed_joint_31: type fixed, parent tibia_1, child foot_1, origin xyz=0.097960 -0.020240 0.000000 rpy=0.000000 -1.570796 0.000000
- added joint fixed_joint_32: type fixed, parent tibia_2, child foot_2, origin xyz=0.097960 0.020241 0.000000 rpy=0.000000 -1.570796 0.000000
- added joint fixed_joint_33: type fixed, parent tibia_3, child foot_3, origin xyz=0.097960 0.020240 0.000000 rpy=0.000000 -1.570796 0.000000
- added joint fixed_joint_34: type fixed, parent tibia_4, child foot_4, origin xyz=0.097960 0.020240 0.000000 rpy=0.000000 -1.570796 0.000000
- added joint fixed_joint_35: type fixed, parent tibia_5, child foot_5, origin xyz=0.097960 0.020240 0.000000 rpy=0.000000 -1.570796 0.000000
- added joint fixed_joint_36: type fixed, parent tibia_6, child foot_6, origin xyz=0.097960 0.020240 0.000000 rpy=0.000000 -1.570796 0.000000

Commit message: Relative file paths updated. Requirements file added

File: meshcat_sim/URDF/URDF4Pin/URDF4Pin.urdf (robot description, URDF)
Before this commit: robot base_link, 25 links, 24 joints
Links:
- link coxa_1: geometry visual mesh filename=file://meshcat_sim/URDF/URDF4Pin/URDF4Pin_coxa_1_vis_1.dae
- link coxa_2: geometry visual mesh filename=file://meshcat_sim/URDF/URDF4Pin/URDF4Pin_coxa_2_vis_1.dae
- link coxa_3: geometry visual mesh filename=file://meshcat_sim/URDF/URDF4Pin/URDF4Pin_coxa_3_vis_1.dae
- link coxa_4: geometry visual mesh filename=file://meshcat_sim/URDF/URDF4Pin/URDF4Pin_coxa_4_vis_1.dae
- link coxa_5: geometry visual mesh filename=file://meshcat_sim/URDF/URDF4Pin/URDF4Pin_coxa_5_vis_1.dae
- link coxa_6: geometry visual mesh filename=file://meshcat_sim/URDF/URDF4Pin/URDF4Pin_coxa_6_vis_1.dae
- link femur_1: geometry visual mesh filename=file://meshcat_sim/URDF/URDF4Pin/URDF4Pin_femur_1_vis_1.dae
- link femur_2: geometry visual mesh filename=file://meshcat_sim/URDF/URDF4Pin/URDF4Pin_femur_2_vis_1.dae
- link femur_3: geometry visual mesh filename=file://meshcat_sim/URDF/URDF4Pin/URDF4Pin_femur_3_vis_1.dae
- link femur_4: geometry visual mesh filename=file://meshcat_sim/URDF/URDF4Pin/URDF4Pin_femur_4_vis_1.dae
- link femur_5: geometry visual mesh filename=file://meshcat_sim/URDF/URDF4Pin/URDF4Pin_femur_5_vis_1.dae
- link femur_6: geometry visual mesh filename=file://meshcat_sim/URDF/URDF4Pin/URDF4Pin_femur_6_vis_1.dae
- link robot_base: geometry visual mesh filename=file://meshcat_sim/URDF/URDF4Pin/URDF4Pin_robot_base_vis_1.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
- link tibia_1: geometry visual mesh filename=file://meshcat_sim/URDF/URDF4Pin/URDF4Pin_tibia_1_vis_1.dae
- link tibia_2: geometry visual mesh filename=file://meshcat_sim/URDF/URDF4Pin/URDF4Pin_tibia_2_vis_1.dae
- link tibia_3: geometry visual mesh filename=file://meshcat_sim/URDF/URDF4Pin/URDF4Pin_tibia_3_vis_1.dae
- link tibia_4: geometry visual mesh filename=file://meshcat_sim/URDF/URDF4Pin/URDF4Pin_tibia_4_vis_1.dae
- link tibia_5: geometry visual mesh filename=file://meshcat_sim/URDF/URDF4Pin/URDF4Pin_tibia_5_vis_1.dae
- link tibia_6: geometry visual mesh filename=file://meshcat_sim/URDF/URDF4Pin/URDF4Pin_tibia_6_vis_1.dae

Commit message: Latest URDF including collision and inertial information added. New files created for handling the same.

File: meshcat_sim/URDF/URDF4Pin/URDF4Pin.urdf (robot description, URDF)
Before this commit: robot base_link, 25 links, 24 joints
Links:
- link coxa_1: geometry visual mesh filename=file://URDF/URDF4Pin/URDF4Pin_coxa_1_vis_1.dae
- link coxa_2: geometry visual mesh filename=file://URDF/URDF4Pin/URDF4Pin_coxa_2_vis_1.dae
- link coxa_3: geometry visual mesh filename=file://URDF/URDF4Pin/URDF4Pin_coxa_3_vis_1.dae
- link coxa_4: geometry visual mesh filename=file://URDF/URDF4Pin/URDF4Pin_coxa_4_vis_1.dae
- link coxa_5: geometry visual mesh filename=file://URDF/URDF4Pin/URDF4Pin_coxa_5_vis_1.dae
- link coxa_6: geometry visual mesh filename=file://URDF/URDF4Pin/URDF4Pin_coxa_6_vis_1.dae
- link femur_1: geometry visual mesh filename=file://URDF/URDF4Pin/URDF4Pin_femur_1_vis_1.dae
- link femur_2: geometry visual mesh filename=file://URDF/URDF4Pin/URDF4Pin_femur_2_vis_1.dae
- link femur_3: geometry visual mesh filename=file://URDF/URDF4Pin/URDF4Pin_femur_3_vis_1.dae
- link femur_4: geometry visual mesh filename=file://URDF/URDF4Pin/URDF4Pin_femur_4_vis_1.dae
- link femur_5: geometry visual mesh filename=file://URDF/URDF4Pin/URDF4Pin_femur_5_vis_1.dae
- link femur_6: geometry visual mesh filename=file://URDF/URDF4Pin/URDF4Pin_femur_6_vis_1.dae
- link robot_base: geometry visual mesh filename=file://URDF/URDF4Pin/URDF4Pin_robot_base_vis_1.dae
- link tibia_1: geometry visual mesh filename=file://URDF/URDF4Pin/URDF4Pin_tibia_1_vis_1.dae
- link tibia_2: geometry visual mesh filename=file://URDF/URDF4Pin/URDF4Pin_tibia_2_vis_1.dae
- link tibia_3: geometry visual mesh filename=file://URDF/URDF4Pin/URDF4Pin_tibia_3_vis_1.dae
- link tibia_4: geometry visual mesh filename=file://URDF/URDF4Pin/URDF4Pin_tibia_4_vis_1.dae
- link tibia_5: geometry visual mesh filename=file://URDF/URDF4Pin/URDF4Pin_tibia_5_vis_1.dae
- link tibia_6: geometry visual mesh filename=file://URDF/URDF4Pin/URDF4Pin_tibia_6_vis_1.dae
