Commit message: Latest version - v2.4 1. Joint torque calculation added, need to double check output 2. New script added to control CoppeliaSim simulation 3. URDF Updated

File: meshcat_sim/URDF/VREP_URDF/URDF4DynamicsSim.urdf (robot description, URDF)
Before this commit: robot HexY, 25 links, 24 joints
Joints:
- removed joint Spherical_joint_01
- removed joint Spherical_joint_02
- removed joint Spherical_joint_03
- removed joint Spherical_joint_04
- removed joint Spherical_joint_05
- removed joint Spherical_joint_06
- added joint Fixed_joint_01: type fixed, parent tibia_1, child endeff_1, origin xyz=0.097930 -0.020250 0.000000 rpy=0.000000 -1.570796 0.000000
- added joint Fixed_joint_02: type fixed, parent tibia_2, child endeff_2, origin xyz=0.097930 0.020248 0.000001 rpy=0.000000 -1.570796 0.000000
- added joint Fixed_joint_03: type fixed, parent tibia_B_3, child endeff_3, origin xyz=0.097930 0.020595 0.000199 rpy=0.000000 -1.570796 0.000000
- added joint Fixed_joint_04: type fixed, parent tibia_4, child endeff_4, origin xyz=0.097930 0.020250 0.000000 rpy=0.000000 -1.570796 0.000000
- added joint Fixed_joint_05: type fixed, parent tibia_5, child endeff_5, origin xyz=0.097930 0.020248 0.000001 rpy=-0.000000 -1.570796 0.000000
- added joint Fixed_joint_06: type fixed, parent tibia_6, child endeff_6, origin xyz=0.097930 0.020248 -0.000001 rpy=-0.000000 -1.570796 0.000000
- joint Revolute_joint_01: limit (none) -> lower=-1.0471975511967 upper=1.0471975511967 effort=0.52 velocity=10.786134777326; type continuous -> revolute
- joint Revolute_joint_02: limit (none) -> lower=-1.0471975511967 upper=1.0471975511967 effort=0.52 velocity=10.786134777326; type continuous -> revolute
- joint Revolute_joint_03: limit (none) -> lower=-1.0471975511967 upper=1.0471975511967 effort=0.52 velocity=10.786134777326; type continuous -> revolute
- joint Revolute_joint_04: limit (none) -> lower=-1.0471975511967 upper=1.0471975511967 effort=0.52 velocity=10.786134777326; type continuous -> revolute
- joint Revolute_joint_05: limit (none) -> lower=-1.0471975511967 upper=1.0471975511967 effort=0.52 velocity=10.786134777326; type continuous -> revolute
- joint Revolute_joint_06: limit (none) -> lower=-1.0471975511967 upper=1.0471975511967 effort=0.52 velocity=10.786134777326; type continuous -> revolute
- joint Revolute_joint_11: limit (none) -> lower=-1.0471975511967 upper=1.0471975511967 effort=0.52 velocity=10.786134777326; type continuous -> revolute
- joint Revolute_joint_12: limit (none) -> lower=-1.0471975511967 upper=1.0471975511967 effort=0.52 velocity=10.786134777326; type continuous -> revolute
- joint Revolute_joint_13: limit (none) -> lower=-1.0471975511967 upper=1.0471975511967 effort=0.52 velocity=10.786134777326; type continuous -> revolute
- joint Revolute_joint_14: limit (none) -> lower=-1.0471975511967 upper=1.0471975511967 effort=0.52 velocity=10.786134777326; type continuous -> revolute
- joint Revolute_joint_15: limit (none) -> lower=-1.0471975511967 upper=1.0471975511967 effort=0.52 velocity=10.786134777326; type continuous -> revolute
- joint Revolute_joint_16: limit (none) -> lower=-1.0471975511967 upper=1.0471975511967 effort=0.52 velocity=10.786134777326; type continuous -> revolute
- joint Revolute_joint_21: limit (none) -> lower=-1.0471975511967 upper=1.0471975511967 effort=0.52 velocity=10.786134777326; type continuous -> revolute
- joint Revolute_joint_22: limit (none) -> lower=-1.0471975511967 upper=1.0471975511967 effort=0.52 velocity=10.786134777326; type continuous -> revolute
- joint Revolute_joint_23: limit (none) -> lower=-1.0471975511967 upper=1.0471975511967 effort=0.52 velocity=10.786134777326; type continuous -> revolute
- joint Revolute_joint_24: limit (none) -> lower=-1.0471975511967 upper=1.0471975511967 effort=0.52 velocity=10.786134777326; type continuous -> revolute
- joint Revolute_joint_25: limit (none) -> lower=-1.0471975511967 upper=1.0471975511967 effort=0.52 velocity=10.786134777326; type continuous -> revolute
- joint Revolute_joint_26: limit (none) -> lower=-1.0471975511967 upper=1.0471975511967 effort=0.52 velocity=10.786134777326; type continuous -> revolute
