Commit message: URDF Updated and other minor changes

File: meshcat_sim/URDF/Physics_Model_Edited_old/Physics Model URDF (Edtd.).urdf (robot description, URDF)
Before this commit: robot HexY, 27 links, 26 joints
Links:
- removed link CAM
- removed link robot_base_inertial
- removed link tibia_3
- added link tibia_B_3, mass 0.034569; collision mesh filename=file://URDF/Physics_Model_Edited/Physics Model URDF (Edtd.)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; collision mesh filename=file://URDF/Physics_Model_Edited/Physics Model URDF (Edtd.)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
- link foot_1: mass 1e-09 -> 1e-06; geometry collision mesh filename=file://URDF/Physics_Model_Edited/Physics Model URDF (Edtd.)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; visual mesh filename=file://URDF/Physics_Model_Edited/Physics Model URDF (Edtd.)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
- link foot_2: mass 1e-09 -> 1e-06; geometry collision mesh filename=file://URDF/Physics_Model_Edited/Physics Model URDF (Edtd.)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; visual mesh filename=file://URDF/Physics_Model_Edited/Physics Model URDF (Edtd.)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
- link foot_3: mass 1e-09 -> 1e-06; geometry collision mesh filename=file://URDF/Physics_Model_Edited/Physics Model URDF (Edtd.)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; visual mesh filename=file://URDF/Physics_Model_Edited/Physics Model URDF (Edtd.)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
- link foot_4: mass 1e-09 -> 1e-06; geometry collision mesh filename=file://URDF/Physics_Model_Edited/Physics Model URDF (Edtd.)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; visual mesh filename=file://URDF/Physics_Model_Edited/Physics Model URDF (Edtd.)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
- link foot_5: mass 1e-09 -> 1e-06; geometry collision mesh filename=file://URDF/Physics_Model_Edited/Physics Model URDF (Edtd.)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; visual mesh filename=file://URDF/Physics_Model_Edited/Physics Model URDF (Edtd.)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
- link foot_6: mass 1e-09 -> 1e-06; geometry collision mesh filename=file://URDF/Physics_Model_Edited/Physics Model URDF (Edtd.)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; visual mesh filename=file://URDF/Physics_Model_Edited/Physics Model URDF (Edtd.)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
- link robot_base: mass None -> 1.588718
Joints:
- removed joint Spherical_joint
- removed joint robot_base_inertial_joint
- joint Revolute_joint_01: origin xyz=0.000000 -0.159210 0.059000 rpy=-3.141593 3.141593 0.000000 -> xyz=0.000000 -0.159210 0.059000 rpy=-3.141593 3.141593 -3.141593
- joint Revolute_joint_11: origin xyz=0.000000 0.047000 0.000000 rpy=0.000000 1.570796 0.000000 -> xyz=0.000000 -0.047000 0.000000 rpy=-3.141593 1.570796 0.000000
- joint Revolute_joint_23: child tibia_3 -> tibia_B_3
- joint Spherical_joint_01: origin xyz=0.097930 0.020250 -0.000000 rpy=0.000000 -1.570796 0.000000 -> xyz=0.097930 0.020250 -0.000000 rpy=3.141593 1.570796 0.000000
- joint Spherical_joint_03: parent tibia_3 -> tibia_B_3
