Commit message: Hexapod v2.5.4 new version init

File: meshcat_sim/URDF/Physics_Model_Edited/Physics Model URDF (Edtd.).urdf (robot description, URDF)
Before this commit: robot HexY, 27 links, 26 joints
Links:
- removed link tibia_3
- added link tibia_B_3, mass 0.034569; collision mesh filename=file://URDF/Physics_Model_Edited/Physics Model URDF (Edtd.)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; collision mesh filename=file://URDF/Physics_Model_Edited/Physics Model URDF (Edtd.)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
Joints:
- joint Revolute_joint_01: origin xyz=0.000000 -0.159210 0.059000 rpy=-3.141593 3.141593 0.000000 -> xyz=0.159210 0.000000 0.059000 rpy=-3.141593 3.141593 1.570796
- joint Revolute_joint_02: origin xyz=0.137880 -0.079600 0.059000 rpy=-3.141593 3.141593 1.047198 -> xyz=0.079600 0.137880 0.059000 rpy=-3.141593 3.141593 2.617994
- joint Revolute_joint_03: origin xyz=0.137880 0.079600 0.059000 rpy=-3.141593 3.141593 2.094395 -> xyz=-0.079600 0.137880 0.059000 rpy=-3.141593 3.141593 -2.617994
- joint Revolute_joint_04: origin xyz=0.000000 0.159210 0.059000 rpy=-3.141593 3.141593 -3.141593 -> xyz=-0.159210 -0.000000 0.059000 rpy=-3.141593 3.141593 -1.570796
- joint Revolute_joint_05: origin xyz=-0.137880 0.079600 0.059000 rpy=-3.141593 3.141593 -2.094395 -> xyz=-0.079600 -0.137880 0.059000 rpy=-3.141593 3.141593 -0.523599
- joint Revolute_joint_06: origin xyz=-0.137880 -0.079600 0.059000 rpy=-3.141593 3.141593 -1.047198 -> xyz=0.079600 -0.137880 0.059000 rpy=-3.141593 3.141593 0.523599
- joint Revolute_joint_11: origin xyz=0.000000 0.047000 0.000000 rpy=0.000000 1.570796 0.000000 -> xyz=0.000000 0.047000 0.000000 rpy=-3.141593 1.570796 0.000000
- joint Revolute_joint_12: origin xyz=0.000002 0.046997 -0.000000 rpy=-0.000000 1.570796 0.000000 -> xyz=0.000002 0.046997 -0.000000 rpy=-3.141593 1.570796 0.000000
- joint Revolute_joint_13: origin xyz=-0.000002 0.046997 0.000000 rpy=-0.000000 1.570796 0.000000 -> xyz=-0.000002 0.046997 0.000000 rpy=-3.141593 1.570796 0.000000
- joint Revolute_joint_14: origin xyz=0.000000 0.047000 0.000000 rpy=0.000000 1.570796 0.000000 -> xyz=0.000000 0.047000 0.000000 rpy=-3.141593 1.570796 0.000000
- joint Revolute_joint_15: origin xyz=0.000002 0.046997 0.000000 rpy=0.000000 1.570796 0.000000 -> xyz=0.000002 0.046997 -0.000000 rpy=-3.141593 1.570796 0.000000
- joint Revolute_joint_16: origin xyz=-0.000002 0.046997 0.000000 rpy=0.000000 1.570796 0.000000 -> xyz=-0.000002 0.046997 0.000000 rpy=-3.141593 1.570796 0.000000
- joint Revolute_joint_21: origin xyz=-0.039460 0.023550 -0.000000 rpy=-3.141593 3.141593 3.141593 -> xyz=-0.039460 -0.023550 0.000000 rpy=-3.141593 3.141593 -3.141593
- joint Revolute_joint_22: origin xyz=-0.039460 0.023557 0.000002 rpy=-3.141593 3.141593 3.141593 -> xyz=-0.039460 -0.023557 -0.000002 rpy=-3.141593 3.141593 -3.141593
- joint Revolute_joint_23: child tibia_3 -> tibia_B_3; origin xyz=-0.039460 0.023211 -0.000202 rpy=-3.141593 3.141593 -3.141593 -> xyz=-0.039460 -0.023211 0.000202 rpy=-3.141593 3.141593 -3.141593
- joint Revolute_joint_24: origin xyz=-0.039460 0.023550 -0.000000 rpy=-3.141593 3.141593 -3.141593 -> xyz=-0.039460 -0.023550 0.000000 rpy=-3.141593 3.141593 -3.141593
- joint Revolute_joint_25: origin xyz=-0.039460 0.023557 0.000002 rpy=-3.141593 3.141593 3.141593 -> xyz=-0.039460 -0.023557 -0.000002 rpy=-3.141593 3.141593 -3.141593
- joint Revolute_joint_26: origin xyz=-0.039460 0.023557 -0.000002 rpy=-3.141593 3.141593 -3.141593 -> xyz=-0.039460 -0.023557 0.000002 rpy=3.141593 3.141593 -3.141593
- joint Spherical_joint: origin xyz=0.049709 0.033902 0.133190 rpy=1.570796 3.141593 0.52359877559 -> xyz=0.026094 0.054217 0.133190 rpy=1.570796 3.141593 1.047198
- joint Spherical_joint_01: origin xyz=0.097930 0.020250 -0.000000 rpy=0.000000 -1.570796 0.000000 -> xyz=0.097930 -0.020250 0.000000 rpy=-3.141593 1.570796 0.000000
- joint Spherical_joint_02: origin xyz=0.097930 0.020248 0.000001 rpy=0.000000 -1.570796 0.000000 -> xyz=0.097930 -0.020248 -0.000001 rpy=-3.141593 1.570796 0.000000
- joint Spherical_joint_03: origin xyz=0.097930 0.020595 0.000199 rpy=0.000000 -1.570796 0.000000 -> xyz=0.097930 -0.020595 -0.000199 rpy=-3.141593 1.570796 0.000000; parent tibia_3 -> tibia_B_3
- joint Spherical_joint_04: origin xyz=0.097930 0.020250 0.000000 rpy=0.000000 -1.570796 0.000000 -> xyz=0.097930 -0.020250 -0.000000 rpy=3.141593 1.570796 0.000000
- joint Spherical_joint_05: origin xyz=0.097930 0.020248 0.000001 rpy=-0.000000 -1.570796 0.000000 -> xyz=0.097930 -0.020248 -0.000001 rpy=3.141593 1.570796 0.000000
- joint Spherical_joint_06: origin xyz=0.097930 0.020248 -0.000001 rpy=-0.000000 -1.570796 0.000000 -> xyz=0.097930 -0.020248 0.000001 rpy=3.141593 1.570796 0.000000
- joint robot_base_inertial_joint: origin xyz=0.000000 -0.000000 0.080147 rpy=-3.141593 3.141593 -3.141593 -> xyz=0.000000 0.000000 0.080147 rpy=-3.141593 3.141593 -1.570796
